File: board/CR1TS1A.kicad_pcb (KiCad board)
At the start: 2 copper layers, 111 x 62 mm, 36 parts, among them K1 RELAY_2, P1 USB_OTG, Q1 MMBT3904, Q2 MMBT3904, Q3 MMBT3904, U1 RT9193, U2 HLK-PM01, U4 ESP-12, U5 CH340G, X1 12MHz

Commit message: WIP
Parts:
- added C8: 47u, Capacitors_SMD:C_0805, F.Cu at (150.0, 105.0)
- added C9: 47u, Capacitors_SMD:C_0805, F.Cu at (150.0, 107.0)
- added REF***: OSHW-Logo_11.4x12mm_SilkScreen, Symbols:OSHW-Logo_11.4x12mm_SilkScreen, F.Cu at (189.0, 87.0)
- moved R2 2.67 mm to (156.0, 108.5), turned to 270 degrees
- moved D2 1.55 mm to (152.5, 109.5)
Routing:
- net VCC: track 132.2 -> 135.7 mm
- net GND: track 47.4 -> 50.7 mm, vias 11 -> 13
- net /LED: track 30.5 -> 28.5 mm
- net Net-(D2-Pad2): track 3.04 -> 2.42 mm
Other:
- board text added: "Address"
- board text removed: "- odstranit med pod antenou - logo OSH - stitek pro adresu - 2x47M vedle ESP"

Commit message: WIP
Other:
- board text added: "CC-BY-SA"
Changed lines of the file:
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@@
     (links 87)
     (no_connects 0)
-    (area 80.714287 72.3 220.85 151.7)
+    (area 83.949999 80.949999 195.050001 143.050001)
     (thickness 1.6)
-    (drawings 48)
+    (drawings 49)
     (tracks 285)
     (zones 0)
@@
       (xy 0.633952 -5.96402) (xy 0.746535 -5.366828)) (layer F.SilkS) (width 0.01))
   )
+  (gr_text CC-BY-SA (at 179 83) (layer F.SilkS)
+    (effects (font (size 1 1) (thickness 0.25)))
+  )
   (gr_text Address (at 184.5 130) (layer B.SilkS)

Commit message: WIP
Parts:
- C1, C2, C3, C4, C5, C6, C7, C8, C9: footprint Capacitors_SMD:C_0805 -> Capacitor_SMD:C_0805_2012Metric
- D1, D3, Q1, Q2, Q3: footprint TO_SOT_Packages_SMD:SOT-23 -> Package_TO_SOT_SMD:SOT-23
- D2: footprint LEDs:LED_0805 -> LED_SMD:LED_0805_2012Metric
- L1, R1, R10, R11, R12, R2, R3, R4, R5, R6, R7, R8, R9: footprint Resistors_SMD:R_0805 -> Resistor_SMD:R_0805_2012Metric
- U1: footprint TO_SOT_Packages_SMD:SOT-23-5 -> Package_TO_SOT_SMD:SOT-23-5
- U5: footprint SMD_Packages:SO-16-N -> Package_SO:SOIC-16_3.9x9.9mm_P1.27mm
- X1: footprint Crystals:Crystal_SMD_SeikoEpson_TSX3225-4pin_3.2x2.5mm -> Oscillator:Oscillator_SMD_EuroQuartz_XO32-4Pin_3.2x2.5mm
Connections:
- D3 pad 1: (no net) -> Net-(D3-Pad1)
- K1 pad 12: (no net) -> Net-(K1-Pad12)
- K1 pad 22: (no net) -> Net-(K1-Pad22)
- P1 pad 4: (no net) -> Net-(P1-Pad4)
- U4 pad 2: (no net) -> /ESP/ADC
- U4 pad 4: (no net) -> /ESP/GPIO16
- U4 pad 5: (no net) -> /ESP/GPIO14
- U4 pad 7: (no net) -> /ESP/GPIO13
- U5 pad 10: (no net) -> Net-(U5-Pad10)
- U5 pad 11: (no net) -> Net-(U5-Pad11)
- U5 pad 12: (no net) -> Net-(U5-Pad12)
- U5 pad 15: (no net) -> Net-(U5-Pad15)
- U5 pad 9: (no net) -> Net-(U5-Pad9)
Other:
- board text added: "11.10.2020 symbol and footprint references updated. PCB needs to be checked and fixed (esp. CH340G)"
